File: capewings.brd (EAGLE design)
At the start: 99.1 x 241.3 mm, 51 parts

Commit message: BOM done.
Parts:
- LED1, LED4, LED7: value (none) -> blue
- LED2, LED5, LED8: value (none) -> green
- LED3, LED6, LED9: value (none) -> vdd_blue
- R2, R33, R5: value 4.75K -> 150
- R3, R34, R6: value 4.75K -> 50
