File: capewings.sch (EAGLE design)
At the start: 51 parts

Commit message: BOM done.
Parts:
- LED1, LED4, LED7: value (none) -> blue; MPN (none) -> HT-193NB-5589
- LED2, LED5, LED8: value (none) -> green; MPN (none) -> LG Q971-KN-1
- LED3, LED6, LED9: value (none) -> vdd_blue; MPN (none) -> VLMB1300-GS08
- P1, P4, P6: MPN (none) -> SSHQ-105-D-10-GT-LF
- P10, P13, P16, P19: MPN (none) -> TSHC-105-D-03-145-GT-LF
- P11, P12, P14, P15, P17, P18, P20, P21: MPN (none) -> TSHC-123-D-03-145-GT-LF
- P2, P3, P5, P7, P8, P9: MPN (none) -> SSHQ-123-D-10-GT-LF
- R2, R33, R5: value 4.75K -> 150; MPN (none) -> 302-150-RC
- R3, R34, R6: value 4.75K -> 50; MPN (none) -> 302-49.9-RC
- R7: MPB 302-60.4-RC -> (none); MPN (none) -> 302-60.4-RC
Other:
- note added: "CapeWings"
- note removed: "Cape Name"
- moved on the sheet: LED1, LED2, LED3, LED4, LED5, LED6, LED7, LED8, LED9, P1, P10, P11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
